Commit message: init

File: gym_pybullet_drones/assets/cf2x.urdf (robot description, URDF)
Before this commit: robot cf2, 6 links, 5 joints
Links:
- added link wheel_back_left_link, mass 0; collision cylinder length=0.02 radius=0.015; visual cylinder length=0.02 radius=0.015
- added link wheel_back_right_link, mass 0; collision cylinder length=0.02 radius=0.015; visual cylinder length=0.02 radius=0.015
- added link wheel_front_left_link, mass 0; collision cylinder length=0.02 radius=0.015; visual cylinder length=0.02 radius=0.015
- added link wheel_front_right_link, mass 0; collision cylinder length=0.02 radius=0.015; visual cylinder length=0.02 radius=0.015
Joints:
- added joint wheel_back_left_joint: type continuous, parent base_link, child wheel_back_left_link, origin xyz=-0.03 0.03 -0.02 rpy=-1.5708 0 0, axis 0 0 1
- added joint wheel_back_right_joint: type continuous, parent base_link, child wheel_back_right_link, origin xyz=-0.03 -0.03 -0.02 rpy=-1.5708 0 0, axis 0 0 1
- added joint wheel_front_left_joint: type continuous, parent base_link, child wheel_front_left_link, origin xyz=0.03 0.03 -0.02 rpy=-1.5708 0 0, axis 0 0 1
- added joint wheel_front_right_joint: type continuous, parent base_link, child wheel_front_right_link, origin xyz=0.03 -0.03 -0.02 rpy=-1.5708 0 0, axis 0 0 1
